File: issue3.kicad_sch (KiCad schematic)
At the start: 206 parts, among them IC1 ULA, IC10 4116, IC11 4116, IC12 4116, IC13 4116, IC14 LM1889, IC15 4532, IC16 4532, IC17 4532, IC18 4532, IC19 4532, IC2 Z80, IC20 4532, IC21 4532, IC22 4532, IC23 LS32, IC24 LS00, IC25 LS157, IC26 LS157, IC3 LS157, IC4 LS157, IC5 ROM, IC6 4116, IC7 4116, IC8 4116, IC9 4116, J7 Barrel_Jack_MountingPin, T1 Transformer_1P_1S, X1 14Mhz, X2 4.43Mhz

Commit message: Updated PCB size & Hole Positions
Updated PCB size & Hole Positions. Added stp's for components.
Parts:
- removed BM1, LL1, LR1, TM1: MountingHole, Mod:MountingHole_3.3mm Spectrum, symbol Mechanical:MountingHole
- removed LM1, RM1, RM2: MountingHole, Mod:MountingHole_5mm Spectrum, symbol Mechanical:MountingHole
